File: PicoFox-PCB/PicoFox-PCB.kicad_sch (KiCad schematic)
At the start: 141 parts, among them J2 Conn_01x03_Pin, J3 Conn_02x10_Counter_Clockwise, J4 Conn_Coaxial_Small, J5 USB-TYPE-C-018 (DEALON), Q1 AO3407A, SW3 SK-12D15-G030, U1 BVA1761, U15 USBLC6-2SC6, U16 BQ21040DBVR, U19 ME6217C33M5G, U2 W25Q128JVS, U3 RP2040, U4 Si5351A-B-GT, Y1 ABM8-272-T3, Y2 TG2016SMN_25.0000M-MCGNNM0

Commit message: Initial commit with SSTV support
This is the initial commit that supports SSTV, and file switching.

Includes first pass of the new badge-style fox for Pacificon - HAS NOT BEEN TESTED YET.

**** THIS CODE CONTAINS A LOT OF AI. PLEASE READ THE README.MD ****

Things changed/added to firmware:
- Add SSTV_ENABLE, SSTV_MODE, and VOICE_ENABLE settings
- Support SSTV-only and alternating voice/SSTV operation
- Decode 320x240 JPEGs directly from flash
- Cycle sstv.jpg, sstv1.jpg, sstv2.jpg, etc.
- Add Robot36 color Y/Cb/Cr encoding
- Use separate 5 kHz audio and 3 kHz SSTV FM deviation
- Optimize Si5351 modulation for 8 kHz / 125 us SSTV timing
- Precompute image color data, sine/PLL lookup tables, and phase increments
- Keep SSTV centered at zero carrier offset
- Protect flash access from USB MSC races
- Remove obsolete test-pattern and experimental timing code
- Add timing-critical code documentation
- Add v35 firmware version reporting to keep track of things for the AI side of the house.
Parts:
- removed H1, H2, H3, H4: MountingHole, MountingHole:MountingHole_2.7mm_M2.5_Pad, symbol Mechanical:MountingHole_Pad
- removed J2: Conn_01x03_Pin, Connector_JST:JST_SH_SM03B-SRSS-TB_1x03-1MP_P1.00mm_Horizontal, symbol Connector:Conn_01x03_Pin
- removed J3: Conn_02x10_Counter_Clockwise, Connector_PinHeader_2.54mm:PinHeader_2x10_P2.54mm_Vertical_SMD, symbol Connector_Generic:Conn_02x10_Odd_Even
- removed JP1, JP2: SolderJumper_2_Open, Jumper:SolderJumper-2_P1.3mm_Open_RoundedPad1.0x1.5mm, symbol Jumper:SolderJumper_2_Open
- removed TP1, TP2, TP3, TP4, TP5, TP6, TP7, TP8, TP9: TestPoint, TestPoint:TestPoint_Pad_D1.0mm, symbol Connector:TestPoint
- removed TP14, TP17, TP19, TP20, TP21, TP22, TP23, TP24, TP25, TP26, TP27, TP28, TP29, TP30, TP31, TP32, TP33, TP34, TP35, TP36, TP37, TP38, TP39, TP40, TP41, TP42, TP43, TP44, TP45, TP46, TP47, TP48, TP49, TP51, TP53: TestPoint, PicofoxLib:Castellation Pad, symbol Connector:TestPoint
- added H1, H2: Lanyard Hole, MountingHole:MountingHole_4.3mm_M4_DIN965, symbol Mechanical:MountingHole
Connections:
- net at C28.1, D1.2 (A2), L6.2: now also J4.1 (In)
Other:
- note removed: "Both jumpers soldered for standalone operation. Desolder for external amp stage. Two jumpers creates isolation & distance between in and out. External amp is expected to ground the stub between jumpers. Ext amp must also provide it's own ESD protection."
- note removed: "External Amp Tie In"
- note removed: "Extra TPs here are intended as solder points for future upgrades. Upgrades can be installed using castellated holes and soldering directly to the back of this PCB."
- note removed: "Extra TPs here are intended as solder points or pogo pin connections on future upgrades."
- note removed: "Ground points for upgrades provide mechanical and electrical connection. Place these around the perimeter of the planned upgrade board footprint."
- note removed: "IOs"
- title: PicoFox - RP2040 Minimal -> PicoFox - RP2040 Pacificon Edition

Commit message: Minor updates
Adding AI6YM firmware with fix for forced format of filesystem. Updated PCB/Gerbers.
Parts:
- SW1, SW2: value ~ -> (none)
